Commit message: PG works
Except it fails due to holes in the scan
Maybe just hackily patch it

File: robots/LoCoBot/locobot_navigation/urdf/box.urdf.xacro (robot description, xacro)
@@ -6,5 +6,5 @@
             <origin xyz="0 0 0.32" rpy="0 0 0"/>
             <geometry>
-              <box size="0.1 0.1 0.5"/>
+              <box size="0.35 0.35 0.5"/>
             </geometry>
         </visual>
@@ -12,5 +12,5 @@
             <origin xyz="0 0 0.32" rpy="0 0 0"/>
             <geometry>
-              <box size="0.1 0.1 0.5"/>
+              <box size="0.35 0.35 0.5"/>
             </geometry>
         </collision>

Commit message: Navigation works with TEB
I tried too long getting it to work with PG, it's slow and unreliable. Using TEB instead.

File: robots/LoCoBot/locobot_navigation/urdf/box.urdf.xacro (robot description, xacro)
@@ -6,5 +6,5 @@
             <origin xyz="0 0 0.32" rpy="0 0 0"/>
             <geometry>
-              <box size="0.35 0.35 0.5"/>
+              <box size="0.01 0.01 0.5"/>
             </geometry>
         </visual>
@@ -12,5 +12,5 @@
             <origin xyz="0 0 0.32" rpy="0 0 0"/>
             <geometry>
-              <box size="0.35 0.35 0.5"/>
+              <box size="0.01 0.01 0.5"/>
             </geometry>
         </collision>
