Commit message: Fix locobot modified urdf
approximately

File: robots/LoCoBot/locobot_description/urdf/interbotix_locobot_description_modified.urdf (robot description, URDF)
Before this commit: robot locobot, 27 links, 26 joints
Joints:
- joint laser_joint: origin xyz=-0.01364 0.0  0.3966 rpy=0 3.14159265359 3.14159265359 -> xyz=-0.2047 0.0  0.384 rpy=0 3.14159265359 3.14159265359

Commit message: Unified under locobot_control/main.launch
working with PIPS planner...kinda.... it crashes (but the scan is bad)
Some leftover "short sight" scan points. Not sure where from, causes
slam_toolbox to place obstacles directly on the robot.

File: robots/LoCoBot/locobot_description/urdf/interbotix_locobot_description_modified.urdf (robot description, URDF)
Before this commit: robot locobot, 27 links, 26 joints
Links:
- link laser: mass None -> 0.3

Commit message: Renormalize scan to be upwards in Z
hopefully this doesn't mess up some mappers which assume this

File: robots/LoCoBot/locobot_description/urdf/interbotix_locobot_description_modified.urdf (robot description, URDF)
Before this commit: robot locobot, 27 links, 26 joints
Links:
- added link laser_upright
Joints:
- added joint flip_laser_joint: type fixed, parent laser, child laser_upright, origin xyz=0.0 0.0 0.0 rpy=3.14159265359 0.0 0.0

Commit message: Add stuff for depth image to laserscan
but it isn't correctly processed by the egocircle
can't do infs (crashes the code) and the current running solution (set to max range) clears laser

File: robots/LoCoBot/locobot_description/urdf/interbotix_locobot_description_modified.urdf (robot description, URDF)
Before this commit: robot locobot, 28 links, 27 joints
Links:
- added link camera_frame
Joints:
- added joint camera_coords: type fixed, parent camera_link, child camera_frame, origin xyz=0 0 0 rpy=-1.57079632679489 0 -1.57079632679489, axis 0 0 0
